File: Kicad/chessconnect.kicad_pcb (KiCad board)
At the start: 2 copper layers, 396.3 x 336.1 mm, 260 parts, among them IC1 SN74LVC125ADR, J1 Screw_Terminal_01x02, J3 AVR-ISP-6, SW8 SW_Push, T1 TestPoint, T10 TestPoint, T11 TestPoint, T12 TestPoint, T13 TestPoint, T14 TestPoint, T15 TestPoint, T16 TestPoint, T17 TestPoint, T18 TestPoint, T19 TestPoint, T2 TestPoint, T20 TestPoint, T21 TestPoint, T22 TestPoint, T23 TestPoint, T24 TestPoint, T25 TestPoint, T26 TestPoint, T27 TestPoint, T28 TestPoint, T29 TestPoint, T3 TestPoint, T30 TestPoint, T31 TestPoint, T32 TestPoint, T33 TestPoint, T34 TestPoint, T35 TestPoint, T36 TestPoint, T37 TestPoint, T38 TestPoint, T39 TestPoint, T4 TestPoint, T40 TestPoint, T41 TestPoint, T42 TestPoint, T43 TestPoint, T44 TestPoint, T45 TestPoint, T46 TestPoint, T47 TestPoint, T48 TestPoint, T49 TestPoint, T5 TestPoint, T50 TestPoint, T51 TestPoint, T52 TestPoint, T53 TestPoint, T54 TestPoint, T55 TestPoint, T56 TestPoint, T57 TestPoint, T58 TestPoint, T59 TestPoint, T6 TestPoint, T60 TestPoint, T61 TestPoint, T62 TestPoint, T63 TestPoint, T64 TestPoint, T7 TestPoint, T8 TestPoint, T9 TestPoint, U1 MPR121QR2, U2 TCA9548APWR, U3 MPR121QR2, U4 ATmega328P-P, U5 MPR121QR2, U6 MPR121QR2, U7 MPR121QR2, U8 MPR121QR2, U9 LM1117DT-3.3, Y1 Crystal

Commit message: correction drc warnings
Routing:
- net /RESET: track 326.4 -> 328.0 mm
- net Net-(U5-ELE2): track 139.5 -> 140.6 mm
- net Net-(U5-ELE0): track 56.7 -> 57.8 mm
- net +3.3V: track 607.6 -> 608.7 mm
- net Net-(U5-ELE1): track 98.3 -> 99.3 mm
- net Net-(U1-LED4/ELE8): track 57.9 -> 58.7 mm
- net Net-(U6-LED4/ELE8): track 227.2 -> 227.9 mm
