File: jlcpcb/assembly/assembly.kicad_pcb (KiCad board)
At the start: 2 copper layers, 254 x 254 mm, 250 parts, among them J2 Conn_01x02_Pin, J3 Conn_01x02_Pin, J5 Conn_01x18_Pin, T1 TestPoint, T10 TestPoint, T11 TestPoint, T12 TestPoint, T13 TestPoint, T14 TestPoint, T15 TestPoint, T16 TestPoint, T2 TestPoint, T3 TestPoint, T4 TestPoint, T5 TestPoint, T6 TestPoint, T7 TestPoint, T8 TestPoint, T9 TestPoint

Commit message: holes change
Parts:
- removed ? (x12): , 
- removed the C1 at (41.0, 100.2)
- removed the C1 at (41.0, 36.1)
- removed the C1 at (41.0, 228.2)
- removed the C1 at (41.0, 164.2)
- removed the C10 at (232.9, 132.2)
- removed the C10 at (232.9, 68.2)
- removed the C10 at (232.9, 260.1)
- removed the C10 at (232.9, 196.2)
- removed the C11 at (200.9, 132.2)
- removed the C11 at (200.9, 68.2)
- removed the C11 at (200.9, 260.2)
- removed the C11 at (200.9, 196.2)
- removed the C12 at (168.9, 132.2)
- removed the C12 at (168.9, 68.2)
- removed the C12 at (168.9, 196.2)
- removed the C12 at (168.9, 260.1)
- removed the C13 at (136.9, 68.2)
- removed the C13 at (136.9, 196.2)
- removed the C13 at (136.9, 260.1)
- removed the C13 at (136.9, 132.2)
- removed the C14 at (104.9, 132.2)
- removed the C14 at (104.9, 196.2)
- removed the C14 at (104.9, 68.2)
- removed the C14 at (104.9, 260.1)
- removed the C15 at (72.9, 132.2)
- removed the C15 at (72.9, 196.2)
- removed the C15 at (72.9, 68.2)
- removed the C15 at (72.9, 260.1)
- removed the C16 at (40.9, 132.2)
- removed the C16 at (40.9, 68.2)
- removed the C16 at (40.9, 196.2)
- removed the C16 at (40.9, 260.1)
- removed the C2 at (72.9, 36.1)
- removed the C2 at (72.9, 164.2)
- removed the C2 at (72.9, 228.2)
- removed the C2 at (72.9, 100.2)
- removed the C3 at (104.9, 36.1)
- removed the C3 at (104.9, 228.2)
- removed the C3 at (104.9, 100.2)
- removed the C3 at (104.9, 164.2)
- removed the C4 at (136.9, 228.2)
- removed the C4 at (136.9, 164.2)
- removed the C4 at (136.9, 36.1)
- removed the C4 at (136.9, 100.2)
- removed the C5 at (168.9, 164.2)
- removed the C5 at (168.9, 36.1)
- removed the C5 at (168.9, 228.2)
- removed the C5 at (168.9, 100.2)
- removed the C6 at (200.9, 36.1)
- removed the C6 at (200.9, 164.2)
- removed the C6 at (200.9, 228.2)
- removed the C6 at (200.9, 100.2)
- removed the C7 at (232.9, 36.1)
- removed the C7 at (232.9, 100.2)
- removed the C7 at (232.9, 228.2)
- removed the C7 at (232.9, 164.2)
- removed the C8 at (264.9, 36.1)
- removed the C8 at (264.9, 100.2)
- removed the C8 at (264.9, 164.2)
- removed the C8 at (264.9, 228.2)
- removed the C9 at (264.9, 68.2)
- removed the C9 at (264.9, 260.1)
- removed the C9 at (264.9, 132.2)
- removed the C9 at (264.9, 196.2)
- removed the D1 at (36.0, 226.5)
- removed the D1 at (36.0, 34.5)
- removed the D1 at (36.0, 162.5)
- removed the D1 at (36.0, 98.5)
- removed the D10 at (228.0, 66.5)
- removed the D10 at (228.0, 194.5)
- removed the D10 at (228.0, 130.5)
- removed the D10 at (228.0, 258.5)
- removed the D11 at (196.0, 194.5)
- removed the D11 at (196.0, 130.5)
- removed the D11 at (196.0, 258.5)
- removed the D11 at (196.0, 66.5)
- removed the D12 at (164.0, 130.5)
- removed the D12 at (164.0, 258.5)
- removed the D12 at (164.0, 66.5)
- removed the D12 at (164.0, 194.5)
- removed the D13 at (132.0, 66.5)
- removed the D13 at (132.0, 258.5)
- removed the D13 at (132.0, 194.5)
- removed the D13 at (132.0, 130.5)
- removed the D14 at (100.0, 258.5)
- removed the D14 at (100.0, 66.5)
- removed the D14 at (100.0, 194.5)
- removed the D14 at (100.0, 130.5)
- removed the D15 at (68.0, 130.5)
- removed the D15 at (68.0, 258.5)
- removed the D15 at (68.0, 194.5)
- removed the D15 at (68.0, 66.5)
- removed the D16 at (36.0, 66.5)
- removed the D16 at (36.0, 130.5)
- removed the D16 at (36.0, 194.5)
- removed the D16 at (36.0, 258.5)
- removed the D2 at (68.0, 98.5)
- removed the D2 at (68.0, 162.5)
- removed the D2 at (68.0, 34.5)
- removed the D2 at (68.0, 226.5)
- removed the D3 at (100.0, 162.5)
- removed the D3 at (100.0, 226.5)
- removed the D3 at (100.0, 34.5)
- removed the D3 at (100.0, 98.5)
- removed the D4 at (132.0, 226.5)
- removed the D4 at (132.0, 98.5)
- removed the D4 at (132.0, 162.5)
- removed the D4 at (132.0, 34.5)
- removed the D5 at (164.0, 162.5)
- removed the D5 at (164.0, 34.5)
- removed the D5 at (164.0, 98.5)
- removed the D5 at (164.0, 226.5)
- removed the D6 at (196.0, 162.5)
- removed the D6 at (196.0, 34.5)
- removed the D6 at (196.0, 226.5)
- removed the D6 at (196.0, 98.5)
- removed the D7 at (228.0, 226.5)
- removed the D7 at (228.0, 98.5)
- removed the D7 at (228.0, 34.5)
- removed the D7 at (228.0, 162.5)
- removed the D8 at (260.0, 226.5)
- removed the D8 at (260.0, 98.5)
- removed the D8 at (260.0, 162.5)
- removed the D8 at (260.0, 34.5)
- removed the D9 at (260.0, 194.5)
- removed the D9 at (260.0, 258.5)
- removed the D9 at (260.0, 66.5)
- removed the D9 at (260.0, 130.5)
- removed the H1 at (26.0, 140.5)
- removed the H1 at (26.0, 76.5)
- removed the H1 at (26.0, 268.5)
- removed the H1 at (26.0, 204.5)
- removed the H2 at (26.0, 152.6)
- removed the H2 at (26.0, 88.6)
- removed the H2 at (26.0, 216.6)
- removed the H2 at (26.0, 24.6)
- removed the H3 at (107.3, 216.7)
- removed the H3 at (107.3, 88.7)
- removed the H3 at (107.3, 152.7)
- removed the H3 at (107.3, 24.7)
- removed the H4 at (107.3, 76.6)
- removed the H4 at (107.3, 140.6)
- removed the H4 at (107.3, 204.6)
- removed the H4 at (107.3, 268.6)
- removed the H5 at (188.6, 152.7)
- removed the H5 at (188.6, 88.7)
- removed the H5 at (188.6, 24.7)
- removed the H5 at (188.6, 216.7)
- removed the H6 at (188.6, 204.7)
- removed the H6 at (188.6, 76.7)
- removed the H6 at (188.6, 268.7)
- removed the H6 at (188.6, 140.7)
- removed the H7 at (270.0, 216.4)
- removed the H7 at (270.0, 152.4)
- removed the H7 at (270.0, 24.4)
- removed the H7 at (270.0, 88.4)
- removed the H8 at (270.0, 140.5)
- removed the H8 at (270.0, 76.5)
- removed the H8 at (270.0, 268.5)
- removed the H8 at (270.0, 204.5)
- removed the J2 at (36.8, 78.6)
- removed the J2 at (36.8, 142.6) (x2)
- removed the J2 at (36.8, 206.6)
- removed the J2 at (36.8, 270.6)
- removed the J3 at (36.8, 150.8) (x2)
- removed the J3 at (36.8, 22.8)
- removed the J3 at (36.8, 214.8)
- removed the J3 at (36.8, 86.8)
- removed the J5 at (267.7, 242.4)
- removed the J5 at (267.7, 178.4)
- removed the J5 at (267.7, 114.4)
- removed the J5 at (267.7, 50.4)
- removed the T1 at (46.8, 45.4)
- removed the T1 at (46.8, 237.4)
- removed the T1 at (46.8, 109.4)
- removed the T1 at (46.8, 173.4)
- removed the T10 at (57.2, 119.7)
- removed the T10 at (57.2, 183.7)
- removed the T10 at (57.2, 55.6)
- removed the T10 at (57.2, 247.7)
- removed the T11 at (110.8, 55.6)
- removed the T11 at (110.8, 247.7)
- removed the T11 at (110.8, 183.7)
- removed the T11 at (110.8, 119.7)
- removed the T12 at (121.2, 183.7)
- removed the T12 at (121.2, 55.6)
- removed the T12 at (121.2, 247.7)
- removed the T12 at (121.2, 119.7)
- removed the T13 at (174.9, 119.7)
- removed the T13 at (174.9, 247.7)
- removed the T13 at (174.9, 183.7)
- removed the T13 at (174.9, 55.6)
- removed the T14 at (185.2, 55.6)
- removed the T14 at (185.2, 247.7)
- removed the T14 at (185.2, 119.7)
- removed the T14 at (185.2, 183.7)
- removed the T15 at (238.8, 183.7)
- removed the T15 at (238.8, 247.7)
- removed the T15 at (238.8, 119.7)
- removed the T15 at (238.8, 55.6)
- removed the T16 at (249.2, 55.5)
- removed the T16 at (249.2, 247.6)
- removed the T16 at (249.2, 119.5)
- removed the T16 at (249.2, 183.6)
- removed the T2 at (57.2, 173.4)
- removed the T2 at (57.2, 109.4)
- removed the T2 at (57.2, 237.4)
- removed the T2 at (57.2, 45.4)
- removed the T3 at (110.9, 45.4)
- removed the T3 at (110.9, 109.4)
- removed the T3 at (110.9, 237.4)
- removed the T3 at (110.9, 173.4)
- removed the T4 at (121.2, 109.4)
- removed the T4 at (121.2, 237.4)
- removed the T4 at (121.2, 45.4)
- removed the T4 at (121.2, 173.4)
- removed the T5 at (174.8, 45.4)
- removed the T5 at (174.8, 109.4)
- removed the T5 at (174.8, 237.4)
- removed the T5 at (174.8, 173.4)
- removed the T6 at (185.2, 173.4)
- removed the T6 at (185.2, 237.4)
- removed the T6 at (185.2, 109.4)
- removed the T6 at (185.2, 45.4)
- removed the T7 at (238.8, 45.4)
- removed the T7 at (238.8, 237.4)
- removed the T7 at (238.8, 173.4)
- removed the T7 at (238.8, 109.4)
- removed the T8 at (249.2, 109.4)
- removed the T8 at (249.2, 45.4)
- removed the T8 at (249.2, 173.4)
- removed the T8 at (249.2, 237.4)
- removed the T9 at (46.8, 247.6)
- removed the T9 at (46.8, 119.5)
- removed the T9 at (46.8, 183.6)
- removed the T9 at (46.8, 55.5)
- added C1: 100p, Capacitor_SMD:C_0402_1005Metric_Pad0.74x0.62mm_HandSolder, F.Cu at (42.0, 166.6)
- added C1: 100p, Capacitor_SMD:C_0402_1005Metric_Pad0.74x0.62mm_HandSolder, F.Cu at (42.0, 38.6)
- added C1: 100p, Capacitor_SMD:C_0402_1005Metric_Pad0.74x0.62mm_HandSolder, F.Cu at (42.0, 230.7)
- added C1: 100p, Capacitor_SMD:C_0402_1005Metric_Pad0.74x0.62mm_HandSolder, F.Cu at (42.0, 102.6)
- added C10: 100p, Capacitor_SMD:C_0402_1005Metric_Pad0.74x0.62mm_HandSolder, F.Cu at (233.9, 134.6)
- added C10: 100p, Capacitor_SMD:C_0402_1005Metric_Pad0.74x0.62mm_HandSolder, F.Cu at (233.9, 70.6)
- added C10: 100p, Capacitor_SMD:C_0402_1005Metric_Pad0.74x0.62mm_HandSolder, F.Cu at (233.9, 262.7)
- added C10: 100p, Capacitor_SMD:C_0402_1005Metric_Pad0.74x0.62mm_HandSolder, F.Cu at (233.9, 198.6)
- added C11: 100p, Capacitor_SMD:C_0402_1005Metric_Pad0.74x0.62mm_HandSolder, F.Cu at (201.9, 198.7)
- added C11: 100p, Capacitor_SMD:C_0402_1005Metric_Pad0.74x0.62mm_HandSolder, F.Cu at (201.9, 70.6)
- added C11: 100p, Capacitor_SMD:C_0402_1005Metric_Pad0.74x0.62mm_HandSolder, F.Cu at (201.9, 262.7)
- added C11: 100p, Capacitor_SMD:C_0402_1005Metric_Pad0.74x0.62mm_HandSolder, F.Cu at (201.9, 134.7)
- added C12: 100p, Capacitor_SMD:C_0402_1005Metric_Pad0.74x0.62mm_HandSolder, F.Cu at (169.9, 198.6)
- added C12: 100p, Capacitor_SMD:C_0402_1005Metric_Pad0.74x0.62mm_HandSolder, F.Cu at (169.9, 70.6)
- added C12: 100p, Capacitor_SMD:C_0402_1005Metric_Pad0.74x0.62mm_HandSolder, F.Cu at (169.9, 262.7)
- added C12: 100p, Capacitor_SMD:C_0402_1005Metric_Pad0.74x0.62mm_HandSolder, F.Cu at (169.9, 134.6)
- added C13: 100p, Capacitor_SMD:C_0402_1005Metric_Pad0.74x0.62mm_HandSolder, F.Cu at (137.9, 198.6)
- added C13: 100p, Capacitor_SMD:C_0402_1005Metric_Pad0.74x0.62mm_HandSolder, F.Cu at (137.9, 134.6)
- added C13: 100p, Capacitor_SMD:C_0402_1005Metric_Pad0.74x0.62mm_HandSolder, F.Cu at (137.9, 262.7)
- added C13: 100p, Capacitor_SMD:C_0402_1005Metric_Pad0.74x0.62mm_HandSolder, F.Cu at (137.9, 70.6)
- added C14: 100p, Capacitor_SMD:C_0402_1005Metric_Pad0.74x0.62mm_HandSolder, F.Cu at (105.9, 70.6)
- added C14: 100p, Capacitor_SMD:C_0402_1005Metric_Pad0.74x0.62mm_HandSolder, F.Cu at (105.9, 134.6)
- added C14: 100p, Capacitor_SMD:C_0402_1005Metric_Pad0.74x0.62mm_HandSolder, F.Cu at (105.9, 198.6)
- added C14: 100p, Capacitor_SMD:C_0402_1005Metric_Pad0.74x0.62mm_HandSolder, F.Cu at (105.9, 262.7)
- added C15: 100p, Capacitor_SMD:C_0402_1005Metric_Pad0.74x0.62mm_HandSolder, F.Cu at (73.9, 198.6)
- added C15: 100p, Capacitor_SMD:C_0402_1005Metric_Pad0.74x0.62mm_HandSolder, F.Cu at (73.9, 262.7)
- added C15: 100p, Capacitor_SMD:C_0402_1005Metric_Pad0.74x0.62mm_HandSolder, F.Cu at (73.9, 134.6)
- added C15: 100p, Capacitor_SMD:C_0402_1005Metric_Pad0.74x0.62mm_HandSolder, F.Cu at (73.9, 70.6)
- added C16: 100p, Capacitor_SMD:C_0402_1005Metric_Pad0.74x0.62mm_HandSolder, F.Cu at (41.9, 262.7)
- added C16: 100p, Capacitor_SMD:C_0402_1005Metric_Pad0.74x0.62mm_HandSolder, F.Cu at (41.9, 198.6)
- added C16: 100p, Capacitor_SMD:C_0402_1005Metric_Pad0.74x0.62mm_HandSolder, F.Cu at (41.9, 134.6)
- added C16: 100p, Capacitor_SMD:C_0402_1005Metric_Pad0.74x0.62mm_HandSolder, F.Cu at (41.9, 70.6)
- added C2: 100p, Capacitor_SMD:C_0402_1005Metric_Pad0.74x0.62mm_HandSolder, F.Cu at (73.9, 38.6)
- added C2: 100p, Capacitor_SMD:C_0402_1005Metric_Pad0.74x0.62mm_HandSolder, F.Cu at (73.9, 166.6)
- added C2: 100p, Capacitor_SMD:C_0402_1005Metric_Pad0.74x0.62mm_HandSolder, F.Cu at (73.9, 230.7)
- added C2: 100p, Capacitor_SMD:C_0402_1005Metric_Pad0.74x0.62mm_HandSolder, F.Cu at (73.9, 102.6)
- added C3: 100p, Capacitor_SMD:C_0402_1005Metric_Pad0.74x0.62mm_HandSolder, F.Cu at (105.9, 102.6)
- added C3: 100p, Capacitor_SMD:C_0402_1005Metric_Pad0.74x0.62mm_HandSolder, F.Cu at (105.9, 38.6)
- added C3: 100p, Capacitor_SMD:C_0402_1005Metric_Pad0.74x0.62mm_HandSolder, F.Cu at (105.9, 230.7)
- added C3: 100p, Capacitor_SMD:C_0402_1005Metric_Pad0.74x0.62mm_HandSolder, F.Cu at (105.9, 166.6)
- added C4: 100p, Capacitor_SMD:C_0402_1005Metric_Pad0.74x0.62mm_HandSolder, F.Cu at (137.9, 230.7)
- added C4: 100p, Capacitor_SMD:C_0402_1005Metric_Pad0.74x0.62mm_HandSolder, F.Cu at (137.9, 102.6)
- added C4: 100p, Capacitor_SMD:C_0402_1005Metric_Pad0.74x0.62mm_HandSolder, F.Cu at (137.9, 166.6)
- added C4: 100p, Capacitor_SMD:C_0402_1005Metric_Pad0.74x0.62mm_HandSolder, F.Cu at (137.9, 38.6)
- added C5: 100p, Capacitor_SMD:C_0402_1005Metric_Pad0.74x0.62mm_HandSolder, F.Cu at (169.9, 38.6)
- added C5: 100p, Capacitor_SMD:C_0402_1005Metric_Pad0.74x0.62mm_HandSolder, F.Cu at (169.9, 102.6)
- added C5: 100p, Capacitor_SMD:C_0402_1005Metric_Pad0.74x0.62mm_HandSolder, F.Cu at (169.9, 166.6)
- added C5: 100p, Capacitor_SMD:C_0402_1005Metric_Pad0.74x0.62mm_HandSolder, F.Cu at (169.9, 230.7)
- added C6: 100p, Capacitor_SMD:C_0402_1005Metric_Pad0.74x0.62mm_HandSolder, F.Cu at (201.9, 166.6)
- added C6: 100p, Capacitor_SMD:C_0402_1005Metric_Pad0.74x0.62mm_HandSolder, F.Cu at (201.9, 38.6)
- added C6: 100p, Capacitor_SMD:C_0402_1005Metric_Pad0.74x0.62mm_HandSolder, F.Cu at (201.9, 230.7)
- added C6: 100p, Capacitor_SMD:C_0402_1005Metric_Pad0.74x0.62mm_HandSolder, F.Cu at (201.9, 102.6)
- added C7: 100p, Capacitor_SMD:C_0402_1005Metric_Pad0.74x0.62mm_HandSolder, F.Cu at (234.0, 166.6)
- added C7: 100p, Capacitor_SMD:C_0402_1005Metric_Pad0.74x0.62mm_HandSolder, F.Cu at (234.0, 38.6)
- added C7: 100p, Capacitor_SMD:C_0402_1005Metric_Pad0.74x0.62mm_HandSolder, F.Cu at (234.0, 102.6)
- added C7: 100p, Capacitor_SMD:C_0402_1005Metric_Pad0.74x0.62mm_HandSolder, F.Cu at (234.0, 230.7)
- added C8: 100p, Capacitor_SMD:C_0402_1005Metric_Pad0.74x0.62mm_HandSolder, F.Cu at (265.9, 102.6)
- added C8: 100p, Capacitor_SMD:C_0402_1005Metric_Pad0.74x0.62mm_HandSolder, F.Cu at (265.9, 166.6)
- added C8: 100p, Capacitor_SMD:C_0402_1005Metric_Pad0.74x0.62mm_HandSolder, F.Cu at (265.9, 230.7)
- added C8: 100p, Capacitor_SMD:C_0402_1005Metric_Pad0.74x0.62mm_HandSolder, F.Cu at (265.9, 38.6)
- added C9: 100p, Capacitor_SMD:C_0402_1005Metric_Pad0.74x0.62mm_HandSolder, F.Cu at (266.0, 262.7)
- added C9: 100p, Capacitor_SMD:C_0402_1005Metric_Pad0.74x0.62mm_HandSolder, F.Cu at (266.0, 134.6)
- added C9: 100p, Capacitor_SMD:C_0402_1005Metric_Pad0.74x0.62mm_HandSolder, F.Cu at (266.0, 70.6)
- added C9: 100p, Capacitor_SMD:C_0402_1005Metric_Pad0.74x0.62mm_HandSolder, F.Cu at (266.0, 198.6)
- added D1: WS2812B, LED_SMD:LED_WS2812B_PLCC4_5.0x5.0mm_P3.2mm, F.Cu at (37.0, 36.9)
- added D1: WS2812B, LED_SMD:LED_WS2812B_PLCC4_5.0x5.0mm_P3.2mm, F.Cu at (37.0, 101.0)
- added D1: WS2812B, LED_SMD:LED_WS2812B_PLCC4_5.0x5.0mm_P3.2mm, F.Cu at (37.1, 229.0)
- added D1: WS2812B, LED_SMD:LED_WS2812B_PLCC4_5.0x5.0mm_P3.2mm, F.Cu at (37.1, 165.0)
- added D10: WS2812B, LED_SMD:LED_WS2812B_PLCC4_5.0x5.0mm_P3.2mm, F.Cu at (229.0, 133.0)
- added D10: WS2812B, LED_SMD:LED_WS2812B_PLCC4_5.0x5.0mm_P3.2mm, F.Cu at (229.1, 197.0)
- added D10: WS2812B, LED_SMD:LED_WS2812B_PLCC4_5.0x5.0mm_P3.2mm, F.Cu at (229.0, 68.9)
- added D10: WS2812B, LED_SMD:LED_WS2812B_PLCC4_5.0x5.0mm_P3.2mm, F.Cu at (229.1, 261.0)
- added D11: WS2812B, LED_SMD:LED_WS2812B_PLCC4_5.0x5.0mm_P3.2mm, F.Cu at (197.1, 261.0)
- added D11: WS2812B, LED_SMD:LED_WS2812B_PLCC4_5.0x5.0mm_P3.2mm, F.Cu at (197.0, 133.0)
- added D11: WS2812B, LED_SMD:LED_WS2812B_PLCC4_5.0x5.0mm_P3.2mm, F.Cu at (197.1, 197.0)
- added D11: WS2812B, LED_SMD:LED_WS2812B_PLCC4_5.0x5.0mm_P3.2mm, F.Cu at (197.0, 68.9)
- added D12: WS2812B, LED_SMD:LED_WS2812B_PLCC4_5.0x5.0mm_P3.2mm, F.Cu at (165.0, 68.9)
- added D12: WS2812B, LED_SMD:LED_WS2812B_PLCC4_5.0x5.0mm_P3.2mm, F.Cu at (165.1, 261.0)
- added D12: WS2812B, LED_SMD:LED_WS2812B_PLCC4_5.0x5.0mm_P3.2mm, F.Cu at (165.0, 133.0)
- added D12: WS2812B, LED_SMD:LED_WS2812B_PLCC4_5.0x5.0mm_P3.2mm, F.Cu at (165.1, 197.0)
- added D13: WS2812B, LED_SMD:LED_WS2812B_PLCC4_5.0x5.0mm_P3.2mm, F.Cu at (133.1, 261.0)
- added D13: WS2812B, LED_SMD:LED_WS2812B_PLCC4_5.0x5.0mm_P3.2mm, F.Cu at (133.0, 68.9)
- added D13: WS2812B, LED_SMD:LED_WS2812B_PLCC4_5.0x5.0mm_P3.2mm, F.Cu at (133.1, 197.0)
- added D13: WS2812B, LED_SMD:LED_WS2812B_PLCC4_5.0x5.0mm_P3.2mm, F.Cu at (133.0, 133.0)
- added D14: WS2812B, LED_SMD:LED_WS2812B_PLCC4_5.0x5.0mm_P3.2mm, F.Cu at (101.1, 261.0)
- added D14: WS2812B, LED_SMD:LED_WS2812B_PLCC4_5.0x5.0mm_P3.2mm, F.Cu at (101.0, 68.9)
- added D14: WS2812B, LED_SMD:LED_WS2812B_PLCC4_5.0x5.0mm_P3.2mm, F.Cu at (101.1, 197.0)
- added D14: WS2812B, LED_SMD:LED_WS2812B_PLCC4_5.0x5.0mm_P3.2mm, F.Cu at (101.0, 133.0)
- added D15: WS2812B, LED_SMD:LED_WS2812B_PLCC4_5.0x5.0mm_P3.2mm, F.Cu at (69.1, 261.0)
- added D15: WS2812B, LED_SMD:LED_WS2812B_PLCC4_5.0x5.0mm_P3.2mm, F.Cu at (69.0, 133.0)
- added D15: WS2812B, LED_SMD:LED_WS2812B_PLCC4_5.0x5.0mm_P3.2mm, F.Cu at (69.1, 197.0)
- added D15: WS2812B, LED_SMD:LED_WS2812B_PLCC4_5.0x5.0mm_P3.2mm, F.Cu at (69.0, 68.9)
- added D16: WS2812B, LED_SMD:LED_WS2812B_PLCC4_5.0x5.0mm_P3.2mm, F.Cu at (37.0, 68.9)
- added D16: WS2812B, LED_SMD:LED_WS2812B_PLCC4_5.0x5.0mm_P3.2mm, F.Cu at (37.0, 133.0)
- added D16: WS2812B, LED_SMD:LED_WS2812B_PLCC4_5.0x5.0mm_P3.2mm, F.Cu at (37.1, 261.0)
- added D16: WS2812B, LED_SMD:LED_WS2812B_PLCC4_5.0x5.0mm_P3.2mm, F.Cu at (37.1, 197.0)
- added D2: WS2812B, LED_SMD:LED_WS2812B_PLCC4_5.0x5.0mm_P3.2mm, F.Cu at (69.0, 101.0)
- added D2: WS2812B, LED_SMD:LED_WS2812B_PLCC4_5.0x5.0mm_P3.2mm, F.Cu at (69.1, 165.0)
- added D2: WS2812B, LED_SMD:LED_WS2812B_PLCC4_5.0x5.0mm_P3.2mm, F.Cu at (69.0, 36.9)
- added D2: WS2812B, LED_SMD:LED_WS2812B_PLCC4_5.0x5.0mm_P3.2mm, F.Cu at (69.1, 229.0)
- added D3: WS2812B, LED_SMD:LED_WS2812B_PLCC4_5.0x5.0mm_P3.2mm, F.Cu at (101.0, 101.0)
- added D3: WS2812B, LED_SMD:LED_WS2812B_PLCC4_5.0x5.0mm_P3.2mm, F.Cu at (101.1, 165.0)
- added D3: WS2812B, LED_SMD:LED_WS2812B_PLCC4_5.0x5.0mm_P3.2mm, F.Cu at (101.0, 36.9)
- added D3: WS2812B, LED_SMD:LED_WS2812B_PLCC4_5.0x5.0mm_P3.2mm, F.Cu at (101.1, 229.0)
- added D4: WS2812B, LED_SMD:LED_WS2812B_PLCC4_5.0x5.0mm_P3.2mm, F.Cu at (133.1, 229.0)
- added D4: WS2812B, LED_SMD:LED_WS2812B_PLCC4_5.0x5.0mm_P3.2mm, F.Cu at (133.0, 101.0)
- added D4: WS2812B, LED_SMD:LED_WS2812B_PLCC4_5.0x5.0mm_P3.2mm, F.Cu at (133.0, 36.9)
- added D4: WS2812B, LED_SMD:LED_WS2812B_PLCC4_5.0x5.0mm_P3.2mm, F.Cu at (133.1, 165.0)
- added D5: WS2812B, LED_SMD:LED_WS2812B_PLCC4_5.0x5.0mm_P3.2mm, F.Cu at (165.1, 165.0)
- added D5: WS2812B, LED_SMD:LED_WS2812B_PLCC4_5.0x5.0mm_P3.2mm, F.Cu at (165.1, 229.0)
- added D5: WS2812B, LED_SMD:LED_WS2812B_PLCC4_5.0x5.0mm_P3.2mm, F.Cu at (165.0, 36.9)
- added D5: WS2812B, LED_SMD:LED_WS2812B_PLCC4_5.0x5.0mm_P3.2mm, F.Cu at (165.0, 101.0)
- added D6: WS2812B, LED_SMD:LED_WS2812B_PLCC4_5.0x5.0mm_P3.2mm, F.Cu at (197.0, 36.9)
- added D6: WS2812B, LED_SMD:LED_WS2812B_PLCC4_5.0x5.0mm_P3.2mm, F.Cu at (197.0, 101.0)
- added D6: WS2812B, LED_SMD:LED_WS2812B_PLCC4_5.0x5.0mm_P3.2mm, F.Cu at (197.1, 229.0)
- added D6: WS2812B, LED_SMD:LED_WS2812B_PLCC4_5.0x5.0mm_P3.2mm, F.Cu at (197.1, 165.0)
- added D7: WS2812B, LED_SMD:LED_WS2812B_PLCC4_5.0x5.0mm_P3.2mm, F.Cu at (229.0, 36.9)
- added D7: WS2812B, LED_SMD:LED_WS2812B_PLCC4_5.0x5.0mm_P3.2mm, F.Cu at (229.1, 229.0)
- added D7: WS2812B, LED_SMD:LED_WS2812B_PLCC4_5.0x5.0mm_P3.2mm, F.Cu at (229.0, 101.0)
- added D7: WS2812B, LED_SMD:LED_WS2812B_PLCC4_5.0x5.0mm_P3.2mm, F.Cu at (229.1, 165.0)
- added D8: WS2812B, LED_SMD:LED_WS2812B_PLCC4_5.0x5.0mm_P3.2mm, F.Cu at (261.0, 101.0)
- added D8: WS2812B, LED_SMD:LED_WS2812B_PLCC4_5.0x5.0mm_P3.2mm, F.Cu at (261.1, 229.0)
- added D8: WS2812B, LED_SMD:LED_WS2812B_PLCC4_5.0x5.0mm_P3.2mm, F.Cu at (261.1, 165.0)
- added D8: WS2812B, LED_SMD:LED_WS2812B_PLCC4_5.0x5.0mm_P3.2mm, F.Cu at (261.0, 36.9)
- added D9: WS2812B, LED_SMD:LED_WS2812B_PLCC4_5.0x5.0mm_P3.2mm, F.Cu at (261.1, 197.0)
- added D9: WS2812B, LED_SMD:LED_WS2812B_PLCC4_5.0x5.0mm_P3.2mm, F.Cu at (261.1, 261.0)
- added D9: WS2812B, LED_SMD:LED_WS2812B_PLCC4_5.0x5.0mm_P3.2mm, F.Cu at (261.0, 68.9)
- added D9: WS2812B, LED_SMD:LED_WS2812B_PLCC4_5.0x5.0mm_P3.2mm, F.Cu at (261.0, 133.0)
- added H1: MountingHole_Pad, MountingHole:MountingHole_3.2mm_M3_Pad, F.Cu at (27.0, 143.0)
- added H1: MountingHole_Pad, MountingHole:MountingHole_3.2mm_M3_Pad, F.Cu at (27.1, 271.0)
- added H1: MountingHole_Pad, MountingHole:MountingHole_3.2mm_M3_Pad, F.Cu at (27.0, 78.9)
- added H1: MountingHole_Pad, MountingHole:MountingHole_3.2mm_M3_Pad, F.Cu at (27.1, 207.0)
- added H2: MountingHole_Pad, MountingHole:MountingHole_3.2mm_M3_Pad, F.Cu at (27.0, 27.1)
- added H2: MountingHole_Pad, MountingHole:MountingHole_3.2mm_M3_Pad, F.Cu at (27.1, 155.2)
- added H2: MountingHole_Pad, MountingHole:MountingHole_3.2mm_M3_Pad, F.Cu at (27.0, 91.2)
- added H2: MountingHole_Pad, MountingHole:MountingHole_3.2mm_M3_Pad, F.Cu at (27.1, 219.2)
- added H3: MountingHole_Pad, MountingHole:MountingHole_3.2mm_M3_Pad, F.Cu at (108.4, 219.2)
- added H3: MountingHole_Pad, MountingHole:MountingHole_3.2mm_M3_Pad, F.Cu at (108.3, 91.2)
- added H3: MountingHole_Pad, MountingHole:MountingHole_3.2mm_M3_Pad, F.Cu at (108.3, 27.1)
- added H3: MountingHole_Pad, MountingHole:MountingHole_3.2mm_M3_Pad, F.Cu at (108.4, 155.2)
- added H4: MountingHole_Pad, MountingHole:MountingHole_3.2mm_M3_Pad, F.Cu at (108.4, 271.1)
- added H4: MountingHole_Pad, MountingHole:MountingHole_3.2mm_M3_Pad, F.Cu at (108.4, 207.1)
- added H4: MountingHole_Pad, MountingHole:MountingHole_3.2mm_M3_Pad, F.Cu at (108.3, 143.1)
- added H4: MountingHole_Pad, MountingHole:MountingHole_3.2mm_M3_Pad, F.Cu at (108.3, 79.0)
- added H5: MountingHole_Pad, MountingHole:MountingHole_3.2mm_M3_Pad, F.Cu at (189.6, 27.1)
- added H5: MountingHole_Pad, MountingHole:MountingHole_3.2mm_M3_Pad, F.Cu at (189.7, 219.2)
- added H5: MountingHole_Pad, MountingHole:MountingHole_3.2mm_M3_Pad, F.Cu at (189.6, 91.2)
- added H5: MountingHole_Pad, MountingHole:MountingHole_3.2mm_M3_Pad, F.Cu at (189.7, 155.2)
- added H6: MountingHole_Pad, MountingHole:MountingHole_3.2mm_M3_Pad, F.Cu at (189.7, 271.2)
- added H6: MountingHole_Pad, MountingHole:MountingHole_3.2mm_M3_Pad, F.Cu at (189.6, 143.2)
- added H6: MountingHole_Pad, MountingHole:MountingHole_3.2mm_M3_Pad, F.Cu at (189.7, 207.2)
- added H6: MountingHole_Pad, MountingHole:MountingHole_3.2mm_M3_Pad, F.Cu at (189.6, 79.1)
- added H7: MountingHole_Pad, MountingHole:MountingHole_3.2mm_M3_Pad, F.Cu at (271.1, 219.2)
- added H7: MountingHole_Pad, MountingHole:MountingHole_3.2mm_M3_Pad, F.Cu at (271.0, 91.2)
- added H7: MountingHole_Pad, MountingHole:MountingHole_3.2mm_M3_Pad, F.Cu at (271.0, 27.1)
- added H7: MountingHole_Pad, MountingHole:MountingHole_3.2mm_M3_Pad, F.Cu at (271.1, 155.2)
- added H8: MountingHole_Pad, MountingHole:MountingHole_3.2mm_M3_Pad, F.Cu at (271.1, 271.0)
- added H8: MountingHole_Pad, MountingHole:MountingHole_3.2mm_M3_Pad, F.Cu at (271.0, 143.0)
- added H8: MountingHole_Pad, MountingHole:MountingHole_3.2mm_M3_Pad, F.Cu at (271.1, 207.0)
- added H8: MountingHole_Pad, MountingHole:MountingHole_3.2mm_M3_Pad, F.Cu at (271.0, 78.9)
- added J2: Conn_01x02_Pin, Connector_PinHeader_2.54mm:PinHeader_1x02_P2.54mm_Vertical, B.Cu at (37.9, 273.1)
- added J2: Conn_01x02_Pin, Connector_PinHeader_2.54mm:PinHeader_1x02_P2.54mm_Vertical, B.Cu at (37.9, 209.1)
- added J2: Conn_01x02_Pin, Connector_PinHeader_2.54mm:PinHeader_1x02_P2.54mm_Vertical, B.Cu at (37.8, 81.0)
- added J2: Conn_01x02_Pin, Connector_PinHeader_2.54mm:PinHeader_1x02_P2.54mm_Vertical, B.Cu at (37.8, 145.1)
- added J3: Conn_01x02_Pin, Connector_PinHeader_2.54mm:PinHeader_1x02_P2.54mm_Vertical, B.Cu at (37.8, 25.2)
- added J3: Conn_01x02_Pin, Connector_PinHeader_2.54mm:PinHeader_1x02_P2.54mm_Vertical, B.Cu at (37.9, 153.3)
- added J3: Conn_01x02_Pin, Connector_PinHeader_2.54mm:PinHeader_1x02_P2.54mm_Vertical, B.Cu at (37.8, 89.3)
- added J3: Conn_01x02_Pin, Connector_PinHeader_2.54mm:PinHeader_1x02_P2.54mm_Vertical, B.Cu at (37.9, 217.3)
- added J5: Conn_01x18_Pin, easyeda2kicad:FPC-SMD_18P-P1.00_XUNPU_FPC-1.0FX-18PWCR-H20, B.Cu at (269.2, 52.8)
- added J5: Conn_01x18_Pin, easyeda2kicad:FPC-SMD_18P-P1.00_XUNPU_FPC-1.0FX-18PWCR-H20, B.Cu at (269.3, 244.9)
- added J5: Conn_01x18_Pin, easyeda2kicad:FPC-SMD_18P-P1.00_XUNPU_FPC-1.0FX-18PWCR-H20, B.Cu at (269.3, 180.9)
- added J5: Conn_01x18_Pin, easyeda2kicad:FPC-SMD_18P-P1.00_XUNPU_FPC-1.0FX-18PWCR-H20, B.Cu at (269.2, 116.9)
- added T1: TestPoint, TestPoint:TestPoint_Pad_4.0x4.0mm, F.Cu at (47.9, 239.9)
- added T1: TestPoint, TestPoint:TestPoint_Pad_4.0x4.0mm, F.Cu at (47.9, 175.9)
- added T1: TestPoint, TestPoint:TestPoint_Pad_4.0x4.0mm, F.Cu at (47.8, 111.9)
- added T1: TestPoint, TestPoint:TestPoint_Pad_4.0x4.0mm, F.Cu at (47.8, 47.8)
- added T10: TestPoint, TestPoint:TestPoint_Pad_4.0x4.0mm, F.Cu at (58.2, 122.1)
- added T10: TestPoint, TestPoint:TestPoint_Pad_4.0x4.0mm, F.Cu at (58.3, 250.2)
- added T10: TestPoint, TestPoint:TestPoint_Pad_4.0x4.0mm, F.Cu at (58.3, 186.1)
- added T10: TestPoint, TestPoint:TestPoint_Pad_4.0x4.0mm, F.Cu at (58.2, 58.1)
- added T11: TestPoint, TestPoint:TestPoint_Pad_4.0x4.0mm, F.Cu at (111.9, 250.2)
- added T11: TestPoint, TestPoint:TestPoint_Pad_4.0x4.0mm, F.Cu at (111.8, 122.1)
- added T11: TestPoint, TestPoint:TestPoint_Pad_4.0x4.0mm, F.Cu at (111.9, 186.1)
- added T11: TestPoint, TestPoint:TestPoint_Pad_4.0x4.0mm, F.Cu at (111.8, 58.1)
- added T12: TestPoint, TestPoint:TestPoint_Pad_4.0x4.0mm, F.Cu at (122.2, 58.1)
- added T12: TestPoint, TestPoint:TestPoint_Pad_4.0x4.0mm, F.Cu at (122.3, 186.1)
- added T12: TestPoint, TestPoint:TestPoint_Pad_4.0x4.0mm, F.Cu at (122.2, 122.1)
- added T12: TestPoint, TestPoint:TestPoint_Pad_4.0x4.0mm, F.Cu at (122.3, 250.2)
- added T13: TestPoint, TestPoint:TestPoint_Pad_4.0x4.0mm, F.Cu at (176.0, 250.2)
- added T13: TestPoint, TestPoint:TestPoint_Pad_4.0x4.0mm, F.Cu at (176.0, 58.1)
- added T13: TestPoint, TestPoint:TestPoint_Pad_4.0x4.0mm, F.Cu at (176.0, 186.1)
- added T13: TestPoint, TestPoint:TestPoint_Pad_4.0x4.0mm, F.Cu at (176.0, 122.1)
- added T14: TestPoint, TestPoint:TestPoint_Pad_4.0x4.0mm, F.Cu at (186.3, 250.2)
- added T14: TestPoint, TestPoint:TestPoint_Pad_4.0x4.0mm, F.Cu at (186.2, 58.1)
- added T14: TestPoint, TestPoint:TestPoint_Pad_4.0x4.0mm, F.Cu at (186.2, 122.1)
- added T14: TestPoint, TestPoint:TestPoint_Pad_4.0x4.0mm, F.Cu at (186.3, 186.1)
- added T15: TestPoint, TestPoint:TestPoint_Pad_4.0x4.0mm, F.Cu at (239.9, 250.2)
- added T15: TestPoint, TestPoint:TestPoint_Pad_4.0x4.0mm, F.Cu at (239.8, 58.1)
- added T15: TestPoint, TestPoint:TestPoint_Pad_4.0x4.0mm, F.Cu at (239.8, 122.1)
- added T15: TestPoint, TestPoint:TestPoint_Pad_4.0x4.0mm, F.Cu at (239.9, 186.1)
- added T16: TestPoint, TestPoint:TestPoint_Pad_4.0x4.0mm, F.Cu at (250.3, 250.1)
- added T16: TestPoint, TestPoint:TestPoint_Pad_4.0x4.0mm, F.Cu at (250.2, 58.0)
- added T16: TestPoint, TestPoint:TestPoint_Pad_4.0x4.0mm, F.Cu at (250.3, 186.0)
- added T16: TestPoint, TestPoint:TestPoint_Pad_4.0x4.0mm, F.Cu at (250.2, 122.0)
- added T2: TestPoint, TestPoint:TestPoint_Pad_4.0x4.0mm, F.Cu at (58.2, 111.9)
- added T2: TestPoint, TestPoint:TestPoint_Pad_4.0x4.0mm, F.Cu at (58.2, 47.8)
- added T2: TestPoint, TestPoint:TestPoint_Pad_4.0x4.0mm, F.Cu at (58.3, 175.9)
- added T2: TestPoint, TestPoint:TestPoint_Pad_4.0x4.0mm, F.Cu at (58.3, 239.9)
- added T3: TestPoint, TestPoint:TestPoint_Pad_4.0x4.0mm, F.Cu at (111.9, 47.8)
- added T3: TestPoint, TestPoint:TestPoint_Pad_4.0x4.0mm, F.Cu at (112.0, 175.9)
- added T3: TestPoint, TestPoint:TestPoint_Pad_4.0x4.0mm, F.Cu at (111.9, 111.9)
- added T3: TestPoint, TestPoint:TestPoint_Pad_4.0x4.0mm, F.Cu at (112.0, 239.9)
- added T4: TestPoint, TestPoint:TestPoint_Pad_4.0x4.0mm, F.Cu at (122.3, 175.9)
- added T4: TestPoint, TestPoint:TestPoint_Pad_4.0x4.0mm, F.Cu at (122.2, 47.8)
- added T4: TestPoint, TestPoint:TestPoint_Pad_4.0x4.0mm, F.Cu at (122.2, 111.9)
- added T4: TestPoint, TestPoint:TestPoint_Pad_4.0x4.0mm, F.Cu at (122.3, 239.9)
- added T5: TestPoint, TestPoint:TestPoint_Pad_4.0x4.0mm, F.Cu at (175.9, 175.9)
- added T5: TestPoint, TestPoint:TestPoint_Pad_4.0x4.0mm, F.Cu at (175.8, 47.8)
- added T5: TestPoint, TestPoint:TestPoint_Pad_4.0x4.0mm, F.Cu at (175.9, 239.9)
- added T5: TestPoint, TestPoint:TestPoint_Pad_4.0x4.0mm, F.Cu at (175.8, 111.9)
- added T6: TestPoint, TestPoint:TestPoint_Pad_4.0x4.0mm, F.Cu at (186.3, 175.9)
- added T6: TestPoint, TestPoint:TestPoint_Pad_4.0x4.0mm, F.Cu at (186.2, 111.9)
- added T6: TestPoint, TestPoint:TestPoint_Pad_4.0x4.0mm, F.Cu at (186.2, 47.8)
- added T6: TestPoint, TestPoint:TestPoint_Pad_4.0x4.0mm, F.Cu at (186.3, 239.9)
- added T7: TestPoint, TestPoint:TestPoint_Pad_4.0x4.0mm, F.Cu at (239.9, 239.9)
- added T7: TestPoint, TestPoint:TestPoint_Pad_4.0x4.0mm, F.Cu at (239.8, 111.9)
- added T7: TestPoint, TestPoint:TestPoint_Pad_4.0x4.0mm, F.Cu at (239.8, 47.8)
- added T7: TestPoint, TestPoint:TestPoint_Pad_4.0x4.0mm, F.Cu at (239.9, 175.9)
- added T8: TestPoint, TestPoint:TestPoint_Pad_4.0x4.0mm, F.Cu at (250.2, 47.8)
- added T8: TestPoint, TestPoint:TestPoint_Pad_4.0x4.0mm, F.Cu at (250.2, 111.9)
- added T8: TestPoint, TestPoint:TestPoint_Pad_4.0x4.0mm, F.Cu at (250.3, 239.9)
- added T8: TestPoint, TestPoint:TestPoint_Pad_4.0x4.0mm, F.Cu at (250.3, 175.9)
- added T9: TestPoint, TestPoint:TestPoint_Pad_4.0x4.0mm, F.Cu at (47.8, 58.0)
- added T9: TestPoint, TestPoint:TestPoint_Pad_4.0x4.0mm, F.Cu at (47.9, 250.1)
- added T9: TestPoint, TestPoint:TestPoint_Pad_4.0x4.0mm, F.Cu at (47.9, 186.0)
- added T9: TestPoint, TestPoint:TestPoint_Pad_4.0x4.0mm, F.Cu at (47.8, 122.0)
Routing:
- net /DOUT2: track 145.2 -> 119.4 mm
- net VCC: track 2456.3 -> 2431.5 mm
- net /DataLEDs: track 79.4 -> 77.5 mm
- removed copper zone on F.Cu, net (none)
Other:
- board size 254 x 254 mm -> 254 x 254.1 mm
