File: jlcpcb/matrice/chessconnect_matrice.kicad_pcb (KiCad board)
At the start: 2 copper layers, 254 x 70.2 mm, 63 parts, among them J2 Conn_01x02_Pin, J3 Conn_01x02_Pin, J5 Conn_01x18_Pin, T1 TestPoint, T10 TestPoint, T11 TestPoint, T12 TestPoint, T13 TestPoint, T14 TestPoint, T15 TestPoint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

Commit message: holes change
Parts:
- H1, H2, H3, H4, H5, H6, H7, H8: footprint MountingHole:MountingHole_2.2mm_M2_Pad -> MountingHole:MountingHole_3.2mm_M3_Pad
- moved H7 0.30 mm to (272.8, 74.3)
- moved H2 0.10 mm to (28.8, 74.3)
Connections:
- J5 pad 19: GND -> (no net)
- J5 pad 20: GND -> (no net)
