File: jlcpcb/uP/chessconnect_uP.kicad_pcb (KiCad board)
At the start: 2 copper layers, 100 x 100 mm, 93 parts, among them J1 Screw_Terminal_01x02, J2 AVR-ISP-6, J3 Conn_01x18_Pin, J4 Conn_01x18_Pin, J5 Conn_01x18_Pin, J6 Conn_01x18_Pin, J7 Conn_01x02_Pin, J8 Conn_01x02_Pin, SW1 SW_Push, U1 ATmega328P-P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

Commit message: holes change
Parts:
- H1, H2, H3, H4: footprint MountingHole:MountingHole_2.2mm_M2_Pad -> MountingHole:MountingHole_3.2mm_M3_DIN965_Pad
- moved H3 5.30 mm to (82.0, 100.0)
