File: jlcpcb/uP/chessconnect_uP.kicad_pcb (KiCad board)
At the start: 2 copper layers, 100 x 100 mm, 93 parts, among them J1 Screw_Terminal_01x02, J2 AVR-ISP-6, J3 Conn_01x18_Pin, J4 Conn_01x18_Pin, J5 Conn_01x18_Pin, J6 Conn_01x18_Pin, J7 Conn_01x02_Pin, J8 Conn_01x02_Pin, SW1 SW_Push, U1 ATmega328P-P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

Commit message: ajout alim
Parts:
- removed J1: Screw_Terminal_01x02, TerminalBlock_Phoenix:TerminalBlock_Phoenix_MKDS-3-2-5.08_1x02_P5.08mm_Horizontal
- added DC1: DC-005-A200, easyeda2kicad:DC-IN-TH_DC-005-A200, F.Cu at (164.8, 55.5)
Connections:
- U1 pad 23: unconnected-(U1-PC0-Pad23) -> /detect_alim
Routing:
- net /detect_alim: track 0.00 -> 58.1 mm, vias 0 -> 1
- net ALIM: track 36.7 -> 33.0 mm
