File: jlcpcb/uP/chessconnect_uP.kicad_sch (KiCad schematic)
At the start: 92 parts, among them J1 Screw_Terminal_01x02, J2 AVR-ISP-6, J3 Conn_01x18_Pin, J4 Conn_01x18_Pin, J5 Conn_01x18_Pin, J6 Conn_01x18_Pin, J7 Conn_01x02_Pin, J8 Conn_01x02_Pin, SW1 SW_Push, U1 ATmega328P-P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

Commit message: ajout alim
Parts:
- removed J1: Screw_Terminal_01x02, TerminalBlock_Phoenix:TerminalBlock_Phoenix_MKDS-3-2-5.08_1x02_P5.08mm_Horizontal, symbol Connector:Screw_Terminal_01x02
- added DC1: DC-005-A200, easyeda2kicad:DC-IN-TH_DC-005-A200, symbol easyeda2kicad:DC-005-A200
Connections:
- net ALIM: now also DC1.1
- net GND: now also DC1.2
- net detect_alim: now reaches U1.23 (PC0)
- net detect_alim: now also DC1.3
- no-connect marks 33 -> 32
